Commit message: 位置修改

File: src/ur_gripper_robot/ur_gripper_gazebo/urdf/ur.xacro (robot description, xacro)
@@ -53,5 +53,5 @@
     <parent link="world"/>
     <child link="base_link"/>
-    <origin xyz="0 0 1" rpy="0 0 0"/>
+    <origin xyz="0 0 0" rpy="0 0 0"/>
   </joint>
   <link name="tool0_controller"/>
